Commit message: feat: add open source reference scene assets

File: src/airos_go2w_description/urdf/go2w_nav_eq.urdf.xacro (robot description, xacro)
@@ -2,4 +2,6 @@
 <robot xmlns:xacro="http://www.ros.org/wiki/xacro" name="unitree_go2w_nav_eq">
   <xacro:arg name="controller_config" default="$(find airos_control)/config/go2w_controllers.yaml"/>
+  <xacro:arg name="visual_profile" default="analytic"/>
+  <xacro:property name="visual_profile" value="$(arg visual_profile)"/>
   <xacro:property name="base_length" value="0.70"/>
   <xacro:property name="base_width" value="0.43"/>
@@ -41,4 +43,12 @@
   <xacro:macro name="wheel" params="prefix x y">
     <link name="${prefix}_wheel_link">
+      <xacro:if value="$(eval '${visual_profile}' == 'reference_mesh')">
+        <visual name="go2w_reference_wheel">
+          <origin xyz="0 0 0" rpy="0 0 0"/>
+          <geometry>
+            <mesh filename="package://airos_go2w_description/meshes/open_source_go2w_reference/${'left_wheel.dae' if y &gt; 0 else 'right_wheel.dae'}" scale="1.0 1.0 1.0"/>
+          </geometry>
+        </visual>
+      </xacro:if>
       <visual>
         <origin xyz="0 0 0" rpy="1.57079632679 0 0"/>
@@ -95,4 +105,12 @@
   <link name="base_footprint"/>
   <link name="base_link">
+    <xacro:if value="$(eval '${visual_profile}' == 'reference_mesh')">
+      <visual name="go2w_reference_base">
+        <origin xyz="0 0 0.015" rpy="0 0 0"/>
+        <geometry>
+          <mesh filename="package://airos_go2w_description/meshes/open_source_go2w_reference/base.dae" scale="1.8 2.6 1.3"/>
+        </geometry>
+      </visual>
+    </xacro:if>
     <visual>
       <origin xyz="0 0 0" rpy="0 0 0"/>
@@ -126,4 +144,12 @@
   <xacro:leg_visual prefix="rr" x="${-wheel_x}" y="${-wheel_y}"/>
   <link name="lidar_link">
+    <xacro:if value="$(eval '${visual_profile}' == 'reference_mesh')">
+      <visual name="mid360_reference_visual">
+        <origin xyz="0 0 -0.035" rpy="0 0 3.14159"/>
+        <geometry>
+          <mesh filename="package://airos_go2w_description/meshes/open_source_go2w_reference/mid-360-scaled.dae" scale="1.0 1.0 1.0"/>
+        </geometry>
+      </visual>
+    </xacro:if>
     <visual>
       <origin xyz="0 0 -0.035" rpy="0 0 0"/>

Commit message: feat: add realistic multilevel Go2W visual demo

File: src/airos_go2w_description/urdf/go2w_nav_eq.urdf.xacro (robot description, xacro)
@@ -148,5 +148,5 @@
         <origin xyz="0 0 -0.035" rpy="0 0 3.14159"/>
         <geometry>
-          <mesh filename="package://airos_go2w_description/meshes/open_source_go2w_reference/mid-360-scaled.dae" scale="1.0 1.0 1.0"/>
+          <mesh filename="package://airos_go2w_description/meshes/open_source_go2w_reference/mid-360-scaled.dae" scale="0.001 0.001 0.001"/>
         </geometry>
       </visual>

Commit message: feat: add terrain-aware multilevel navigation demo

File: src/airos_go2w_description/urdf/go2w_nav_eq.urdf.xacro (robot description, xacro)
@@ -5,13 +5,13 @@
   <xacro:property name="visual_profile" value="$(arg visual_profile)"/>
   <xacro:property name="base_length" value="0.70"/>
-  <xacro:property name="base_width" value="0.43"/>
-  <xacro:property name="base_height" value="0.24"/>
-  <xacro:property name="base_z" value="0.24"/>
+  <xacro:property name="base_width" value="0.50"/>
+  <xacro:property name="base_height" value="0.18"/>
+  <xacro:property name="base_z" value="0.18"/>
   <xacro:property name="wheel_radius" value="0.09"/>
   <xacro:property name="wheel_width" value="0.055"/>
   <xacro:property name="wheel_x" value="0.255"/>
-  <xacro:property name="wheel_y" value="0.255"/>
+  <xacro:property name="wheel_y" value="0.36"/>
   <xacro:property name="wheel_z" value="0.095"/>
-  <xacro:property name="body_mass" value="16.0"/>
+  <xacro:property name="body_mass" value="14.0"/>
   <xacro:property name="wheel_mass" value="0.5"/>
   <xacro:macro name="box_inertial" params="mass x y z">
@@ -264,21 +264,21 @@
   <gazebo reference="fl_wheel_link">
     <material>Gazebo/Black</material>
-    <mu1>1.0</mu1>
-    <mu2>1.0</mu2>
+    <mu1>3.0</mu1>
+    <mu2>3.0</mu2>
   </gazebo>
   <gazebo reference="fr_wheel_link">
     <material>Gazebo/Black</material>
-    <mu1>1.0</mu1>
-    <mu2>1.0</mu2>
+    <mu1>3.0</mu1>
+    <mu2>3.0</mu2>
   </gazebo>
   <gazebo reference="rl_wheel_link">
     <material>Gazebo/Black</material>
-    <mu1>1.0</mu1>
-    <mu2>1.0</mu2>
+    <mu1>3.0</mu1>
+    <mu2>3.0</mu2>
   </gazebo>
   <gazebo reference="rr_wheel_link">
     <material>Gazebo/Black</material>
-    <mu1>1.0</mu1>
-    <mu2>1.0</mu2>
+    <mu1>3.0</mu1>
+    <mu2>3.0</mu2>
   </gazebo>
   <gazebo reference="imu_link">

Commit message: Hide analytic robot visuals for mesh profile

File: src/airos_go2w_description/urdf/go2w_nav_eq.urdf.xacro (robot description, xacro)
@@ -51,13 +51,15 @@
         </visual>
       </xacro:if>
-      <visual>
-        <origin xyz="0 0 0" rpy="1.57079632679 0 0"/>
-        <geometry>
-          <cylinder radius="${wheel_radius}" length="${wheel_width}"/>
-        </geometry>
-        <material name="wheel_black">
-          <color rgba="0.015 0.015 0.018 1.0"/>
-        </material>
-      </visual>
+      <xacro:if value="$(eval '${visual_profile}' != 'reference_mesh')">
+        <visual>
+          <origin xyz="0 0 0" rpy="1.57079632679 0 0"/>
+          <geometry>
+            <cylinder radius="${wheel_radius}" length="${wheel_width}"/>
+          </geometry>
+          <material name="wheel_black">
+            <color rgba="0.015 0.015 0.018 1.0"/>
+          </material>
+        </visual>
+      </xacro:if>
       <collision>
         <origin xyz="0 0 0" rpy="1.57079632679 0 0"/>
@@ -113,13 +115,15 @@
       </visual>
     </xacro:if>
-    <visual>
-      <origin xyz="0 0 0" rpy="0 0 0"/>
-      <geometry>
-        <box size="${base_length} ${base_width} ${base_height}"/>
-      </geometry>
-      <material name="body_dark_blue">
-        <color rgba="0.76 0.78 0.78 1.0"/>
-      </material>
-    </visual>
+    <xacro:if value="$(eval '${visual_profile}' != 'reference_mesh')">
+      <visual>
+        <origin xyz="0 0 0" rpy="0 0 0"/>
+        <geometry>
+          <box size="${base_length} ${base_width} ${base_height}"/>
+        </geometry>
+        <material name="body_dark_blue">
+          <color rgba="0.76 0.78 0.78 1.0"/>
+        </material>
+      </visual>
+    </xacro:if>
     <collision>
       <origin xyz="0 0 0" rpy="0 0 0"/>
@@ -139,8 +143,10 @@
   <xacro:wheel prefix="rl" x="${-wheel_x}" y="${wheel_y}"/>
   <xacro:wheel prefix="rr" x="${-wheel_x}" y="${-wheel_y}"/>
-  <xacro:leg_visual prefix="fl" x="${wheel_x}" y="${wheel_y}"/>
-  <xacro:leg_visual prefix="fr" x="${wheel_x}" y="${-wheel_y}"/>
-  <xacro:leg_visual prefix="rl" x="${-wheel_x}" y="${wheel_y}"/>
-  <xacro:leg_visual prefix="rr" x="${-wheel_x}" y="${-wheel_y}"/>
+  <xacro:if value="$(eval '${visual_profile}' != 'reference_mesh')">
+    <xacro:leg_visual prefix="fl" x="${wheel_x}" y="${wheel_y}"/>
+    <xacro:leg_visual prefix="fr" x="${wheel_x}" y="${-wheel_y}"/>
+    <xacro:leg_visual prefix="rl" x="${-wheel_x}" y="${wheel_y}"/>
+    <xacro:leg_visual prefix="rr" x="${-wheel_x}" y="${-wheel_y}"/>
+  </xacro:if>
   <link name="lidar_link">
     <xacro:if value="$(eval '${visual_profile}' == 'reference_mesh')">
@@ -152,13 +158,15 @@
       </visual>
     </xacro:if>
-    <visual>
-      <origin xyz="0 0 -0.035" rpy="0 0 0"/>
-      <geometry>
-        <cylinder radius="0.045" length="0.055"/>
-      </geometry>
-      <material name="sensor_green">
-        <color rgba="0.05 0.50 0.38 1.0"/>
-      </material>
-    </visual>
+    <xacro:if value="$(eval '${visual_profile}' != 'reference_mesh')">
+      <visual>
+        <origin xyz="0 0 -0.035" rpy="0 0 0"/>
+        <geometry>
+          <cylinder radius="0.045" length="0.055"/>
+        </geometry>
+        <material name="sensor_green">
+          <color rgba="0.05 0.50 0.38 1.0"/>
+        </material>
+      </visual>
+    </xacro:if>
     <xacro:cylinder_inertial mass="0.2" radius="0.045" length="0.055"/>
   </link>
@@ -175,13 +183,15 @@
   </joint>
   <link name="imu_link">
-    <visual>
-      <origin xyz="0 0 0" rpy="0 0 0"/>
-      <geometry>
-        <box size="0.055 0.035 0.02"/>
-      </geometry>
-      <material name="imu_orange">
-        <color rgba="0.8 0.35 0.05 1.0"/>
-      </material>
-    </visual>
+    <xacro:if value="$(eval '${visual_profile}' != 'reference_mesh')">
+      <visual>
+        <origin xyz="0 0 0" rpy="0 0 0"/>
+        <geometry>
+          <box size="0.055 0.035 0.02"/>
+        </geometry>
+        <material name="imu_orange">
+          <color rgba="0.8 0.35 0.05 1.0"/>
+        </material>
+      </visual>
+    </xacro:if>
     <collision>
       <origin xyz="0 0 0" rpy="0 0 0"/>
@@ -198,13 +208,15 @@
   </joint>
   <link name="camera_link">
-    <visual>
-      <origin xyz="0 0 0" rpy="0 0 0"/>
-      <geometry>
-        <box size="0.055 0.08 0.045"/>
-      </geometry>
-      <material name="camera_gray">
-        <color rgba="0.18 0.18 0.2 1.0"/>
-      </material>
-    </visual>
+    <xacro:if value="$(eval '${visual_profile}' != 'reference_mesh')">
+      <visual>
+        <origin xyz="0 0 0" rpy="0 0 0"/>
+        <geometry>
+          <box size="0.055 0.08 0.045"/>
+        </geometry>
+        <material name="camera_gray">
+          <color rgba="0.18 0.18 0.2 1.0"/>
+        </material>
+      </visual>
+    </xacro:if>
     <collision>
       <origin xyz="0 0 0" rpy="0 0 0"/>
